Commit message: working GNN V1

File: morpho_gnn_robot/anymal.urdf (robot description, URDF)
Before this commit: robot anymal, 22 links, 21 joints
Links:
- link LF_FOOT: mass None -> 0.3
- link LH_FOOT: mass None -> 0.3
- link RF_FOOT: mass None -> 0.3
- link RH_FOOT: mass None -> 0.3
- link base: mass None -> 15
