Commit message: chore: purge build artifacts, weights, and logs from tracking

File: morpho_gnn_robot/Training_MLP/anymal_stripped.urdf (robot description, URDF)
Before this commit: robot anymal, 33 links, 32 joints
Links:
- removed link LM_ADAPTER
- removed link LM_FOOT
- removed link LM_HIP
- removed link LM_SHANK
- removed link LM_THIGH
- removed link RM_ADAPTER
- removed link RM_FOOT
- removed link RM_HIP
- removed link RM_SHANK
- removed link RM_THIGH
Joints:
- removed joint LM_ADAPTER_TO_FOOT
- removed joint LM_HAA
- removed joint LM_HFE
- removed joint LM_KFE
- removed joint LM_SHANK_TO_ADAPTER
- removed joint RM_ADAPTER_TO_FOOT
- removed joint RM_HAA
- removed joint RM_HFE
- removed joint RM_KFE
- removed joint RM_SHANK_TO_ADAPTER
