Commit message: fix: File paths

File: kaggle_gnn_finetune/kaggle_package/aliengo_stripped.urdf (robot description, URDF)
Before this commit: robot aliengo, 31 links, 30 joints
Links:
- link base: mass None -> 1.0

File: kaggle_gnn_finetune/kaggle_package/go1_stripped.urdf (robot description, URDF)
Before this commit: robot go1, 46 links, 45 joints
Links:
- link base: mass None -> 1.0
- link camera_laserscan_link_left: mass None -> 1.0
- link camera_laserscan_link_right: mass None -> 1.0
- link camera_optical_chin: mass None -> 1.0
- link camera_optical_face: mass None -> 1.0
- link camera_optical_left: mass None -> 1.0
- link camera_optical_rearDown: mass None -> 1.0
- link camera_optical_right: mass None -> 1.0

File: morpho_gnn_robot/Training_Location/anymal.urdf (robot description, URDF)
Before this commit: robot anymal, 23 links, 22 joints
Links:
- link LF_ADAPTER: geometry collision cylinder length=0.32125 radius=0.015; visual mesh filename=../morpho_ros2_ws/src/morpho_robot/meshes/anymal_foot.dae scale=0.001 0.001 0.001
- link LF_HIP: geometry collision cylinder length=0.03 radius=0.045; collision cylinder length=0.1 radius=0.08
- link LF_SHANK: geometry collision box size=0.08 0.07 0.13; visual mesh filename=../morpho_ros2_ws/src/morpho_robot/meshes/anymal_shank_l.dae scale=0.001 0.001 0.001
- link LF_THIGH: geometry collision box size=0.08 0.04 0.25; collision cylinder length=0.12 radius=0.06
- link LH_ADAPTER: geometry collision cylinder length=0.32125 radius=0.015; visual mesh filename=../morpho_ros2_ws/src/morpho_robot/meshes/anymal_foot.dae scale=0.001 0.001 0.001
- link LH_HIP: geometry collision cylinder length=0.03 radius=0.045; collision cylinder length=0.1 radius=0.08
- link LH_SHANK: geometry collision box size=0.08 0.07 0.13; visual mesh filename=../morpho_ros2_ws/src/morpho_robot/meshes/anymal_shank_r.dae scale=0.001 0.001 0.001
- link LH_THIGH: geometry collision box size=0.08 0.04 0.25; collision cylinder length=0.12 radius=0.06
- link RF_ADAPTER: geometry collision cylinder length=0.32125 radius=0.015; visual mesh filename=../morpho_ros2_ws/src/morpho_robot/meshes/anymal_foot.dae scale=0.001 0.001 0.001
- link RF_HIP: geometry collision cylinder length=0.03 radius=0.045; collision cylinder length=0.1 radius=0.08
- link RF_SHANK: geometry collision box size=0.08 0.07 0.13; visual mesh filename=../morpho_ros2_ws/src/morpho_robot/meshes/anymal_shank_r.dae scale=0.001 0.001 0.001
- link RF_THIGH: geometry collision box size=0.08 0.04 0.25; collision cylinder length=0.12 radius=0.06
- link RH_ADAPTER: geometry collision cylinder length=0.32125 radius=0.015; visual mesh filename=../morpho_ros2_ws/src/morpho_robot/meshes/anymal_foot.dae scale=0.001 0.001 0.001
- link RH_HIP: geometry collision cylinder length=0.03 radius=0.045; collision cylinder length=0.1 radius=0.08
- link RH_SHANK: geometry collision box size=0.08 0.07 0.13; visual mesh filename=../morpho_ros2_ws/src/morpho_robot/meshes/anymal_shank_l.dae scale=0.001 0.001 0.001
- link RH_THIGH: geometry collision box size=0.08 0.04 0.25; collision cylinder length=0.12 radius=0.06
- link base: geometry collision box size=0.1 0.1 0.07; collision box size=0.1 0.1 0.07
